Commit message: Adding Diff Drive

File: description/robot.urdf.xacro (robot description, xacro)
@@ -2,3 +2,4 @@
 <robot xmlns:xacro="http://www.ros.org/wiki/xacro"  name="robot">
     <xacro:include filename="robot_base.xacro"/>
+    <xacro:include filename="gazebo_control.xacro"/>
 </robot>

File: description/robot_base.xacro (robot description, xacro)
@@ -57,4 +57,7 @@
         </xacro:inertial_box>
     </link>
+    <gazebo reference="chassis">
+        <material>Gazebo/Orange</material>
+    </gazebo>
     <!-- LEFT WHEEL LINK-->
     <joint name="left_wheel_joint" type="continuous">
@@ -67,5 +70,5 @@
         <visual>
             <geometry>
-                <cylinder radius="0.04" length="0.015"/>
+                <cylinder radius="0.03" length="0.015"/>
             </geometry>
             <material name="blue"/>
@@ -73,11 +76,14 @@
         <collision>
             <geometry>
-                <cylinder radius="0.04" length="0.015"/>
+                <cylinder radius="0.03" length="0.015"/>
             </geometry>
         </collision>
-        <xacro:inertial_cylinder mass="0.1" length="0.015" radius="0.04">
+        <xacro:inertial_cylinder mass="0.1" length="0.015" radius="0.03">
             <origin xyz="0.0 0.0 0.0" rpy="0.0 0.0 0.0"/>
         </xacro:inertial_cylinder>
     </link>
+    <gazebo reference="left_wheel">
+        <material>Gazebo/Blue</material>
+    </gazebo>
     <!-- RIGHT WHEEL LINK-->
     <joint name="right_wheel_joint" type="continuous">
@@ -90,5 +96,5 @@
         <visual>
             <geometry>
-                <cylinder radius="0.04" length="0.015"/>
+                <cylinder radius="0.03" length="0.015"/>
             </geometry>
             <material name="blue"/>
@@ -96,11 +102,14 @@
         <collision>
             <geometry>
-                <cylinder radius="0.04" length="0.015"/>
+                <cylinder radius="0.03" length="0.015"/>
             </geometry>
         </collision>
-        <xacro:inertial_cylinder mass="0.1" length="0.015" radius="0.04">
+        <xacro:inertial_cylinder mass="0.1" length="0.015" radius="0.03">
             <origin xyz="0.0 0.0 0.0" rpy="0.0 0.0 0.0"/>
         </xacro:inertial_cylinder>
     </link>
+    <gazebo reference="right_wheel">
+        <material>Gazebo/Blue</material>
+    </gazebo>
     <!-- CASTER WHEEL LINK -->
     <joint name="caster_wheel_joint" type="fixed">
@@ -112,5 +121,5 @@
         <visual>
             <geometry>
-                <sphere radius="0.04"/>
+                <sphere radius="0.03"/>
             </geometry>
             <material name="white"/>
@@ -118,10 +127,15 @@
         <collision>
             <geometry>
-                <sphere radius="0.04"/>
+                <sphere radius="0.03"/>
             </geometry>
         </collision>
-        <xacro:inertial_sphere mass="0.1" radius="0.04">
+        <xacro:inertial_sphere mass="0.1" radius="0.03">
             <origin xyz="0.0 0.0 0.0" rpy="0.0 0.0 0.0"/>
         </xacro:inertial_sphere>
     </link>
+    <gazebo reference="caster_wheel">
+        <material>Gazebo/White</material>
+        <mu1 value="0.001"/>
+        <mu2 value="0.001"/>
+    </gazebo>
 </robot>

Commit message: Nav2 Capabilities Added

File: description/robot.urdf.xacro (robot description, xacro)
@@ -3,3 +3,4 @@
     <xacro:include filename="robot_base.xacro"/>
     <xacro:include filename="gazebo_control.xacro"/>
+    <xacro:include filename="lidar.xacro"/>
 </robot>

File: description/robot_base.xacro (robot description, xacro)
@@ -31,5 +31,14 @@
         <color rgba="1 0 0 1"/>
     </material>
+    <!-- BASE LINK -->
     <link name="base_link">
+    </link>
+    <!-- BASE_FOOTPRINT LINK -->
+    <joint name="base_footprint_joint" type="fixed">
+        <origin xyz="0.0 0.0 0.0" rpy="0.0 0.0 0.0"/>
+        <parent link="base_link"/>
+        <child link="base_footprint"/>
+    </joint>
+    <link name="base_footprint">
     </link>
     <!-- CHASSIS LINK -->
